File: retro_laptop_musicbox.kicad_pcb (KiCad board)
At the start: 2 copper layers, 260 x 81.6 mm, 80 parts, among them J1 12V Input Barrel, J10 SCREEN, J11 ENCODER, J2 DB25_Male_MountingHoles, J3 MIDI IN, J4 Main Board Connector, J5 DB25_Male_MountingHoles, J6 Jack_3.5mm_5pin, J7 Jack_3.5mm_5pin, J8 Faceplate connector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

Commit message: Update retro_laptop_musicbox.kicad_pcb
Other:
- board text added: "Retro Laptop Musicbox ver. 0.2 2022-2023 https://github.com/madcatse/Retro-laptop-musicbox Using: https://github.com/yeokm1/pcb-covox https://github.com/eigenco/LPT2MIDI https://github.com/chris-jh/mt32-pi-midi-hat"
- board text removed: "Retro Laptop Musicbox ver. 0.2 2022-2023 Using: https://github.com/yeokm1/pcb-covox https://github.com/eigenco/LPT2MIDI https://github.com/chris-jh/mt32-pi-midi-hat"
Changed lines of the file:
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@@
     (effects (font (size 1 1) (thickness 0.15)))
   )
-  (gr_text "Retro Laptop Musicbox ver. 0.2\n2022-2023\nUsing:\nhttps://github.com/yeokm1/pcb-covox\nhttps://github.com/eigenco/LPT2MIDI\nhttps://github.com/chris-jh/mt32-pi-midi-hat" (at 174.7951 76.73) (layer "F.SilkS")
+  (gr_text "Retro Laptop Musicbox ver. 0.2\n2022-2023\nhttps://github.com/madcatse/Retro-laptop-musicbox\nUsing:\nhttps://github.com/yeokm1/pcb-covox\nhttps://github.com/eigenco/LPT2MIDI\nhttps://github.com/chris-jh/mt32-pi-midi-hat" (at 174.7951 78.74) (layer "F.SilkS")
     (effects (font (size 1 1) (thickness 0.15) italic) (justify left))
   )
