File: retro_laptop_musicbox.kicad_sch (KiCad schematic)
At the start: 72 parts, among them J1 12V Input Barrel, J10 SCREEN, J11 ENCODER, J2 DB25_Male_MountingHoles, J3 MIDI IN, J4 Main Board Connector, J5 DB25_Male_MountingHoles, J6 Jack_3.5mm_5pin, J7 Jack_3.5mm_5pin, J8 Faceplate connector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

Commit message: March 26th Update
Other:
- company: (none) -> МИЭТ
- title: Midi/Covox Эмулятор -> MIDI ЭМУЛЯТОР
Changed lines of the file:
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@@
   (paper "A3")
   (title_block
-    (title "Midi/Covox Эмулятор")
+    (title "MIDI ЭМУЛЯТОР")
     (date "2023-03-07")
+    (company "МИЭТ")
     (comment 1 "АЕСН.123456.001")
-    (comment 2 "Панкратова")
+    (comment 2 "Понкратова")
     (comment 3 "Евстафьев")
   )
